Commit message: Complete barebones demo functionality

File: generated_projects/SimpleSim_Example/SimpleSim_Example.urdf/SimpleSim_Example.urdf (robot description, URDF)
Before this commit: robot SimpleSim_Example, 2 links, 1 joints
Links:
- removed link Elevator_Base
- added link Base, mass 6.651333708331838; collision mesh filename=../meshes/Base.stl; visual mesh filename=../meshes/Base.stl
- link Carriage: mass 1.9031493208779748 -> 1.255656511801627
Joints:
- removed joint Elevator_Joint
- added joint Elevator: type prismatic, parent Base, child Carriage, origin xyz=-0.004067949596099795 -0.0038826359001646648 0.347052019548392 rpy=0 0 0, axis 0.0 0.0 1.0, limit lower=-0.3 upper=1.0 effort=100.0 velocity=10.0

File: generated_urdfs/SimpleSim_Example.urdf (robot description, URDF)
Before this commit: robot SimpleSim_Example, 2 links, 1 joints
Links:
- removed link Elevator_Base
- added link Base, mass 6.651333708331838; collision mesh filename=../generated_projects/SimpleSim_Example/meshes/Base.stl; visual mesh filename=../generated_projects/SimpleSim_Example/meshes/Base.stl
- link Carriage: mass 1.9031493208779748 -> 1.255656511801627
Joints:
- removed joint Elevator_Joint
- added joint Elevator: type prismatic, parent Base, child Carriage, origin xyz=-0.004067949596099795 -0.0038826359001646648 0.347052019548392 rpy=0 0 0, axis 0.0 0.0 1.0, limit lower=-0.3 upper=0.8 effort=150.0 velocity=10.0

Commit message: Implement complete visual overhaul

File: generated_projects/SimpleSim_Example/SimpleSim_Example.urdf/SimpleSim_Example.urdf (robot description, URDF)
Before this commit: robot SimpleSim_Example, 2 links, 1 joints
Links:
- link Base: mass 6.651333708331838 -> 5.095193188971689
- link Carriage: mass 1.255656511801627 -> 1.06836643263247
Joints:
- joint Elevator: limit lower=-0.3 upper=1.0 effort=100.0 velocity=10.0 -> lower=-1.0 upper=1.0 effort=100.0 velocity=10.0; origin xyz=-0.004067949596099795 -0.0038826359001646648 0.347052019548392 rpy=0 0 0 -> xyz=-0.0013205222074060543 0.00696341199608074 0.4375544837275319 rpy=0 0 0

File: generated_urdfs/SimpleSim_Example.urdf (robot description, URDF)
Before this commit: robot SimpleSim_Example, 2 links, 1 joints
Links:
- link Base: geometry collision mesh filename=../projects_data/190d5889-94f3-4fcb-8735-7b16cd9e7a9b/meshe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; visual mesh filename=../projects_data/190d5889-94f3-4fcb-8735-7b16cd9e7a9b/meshe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
- link Carriage: geometry collision mesh filename=../projects_data/190d5889-94f3-4fcb-8735-7b16cd9e7a9b/meshe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; visual mesh filename=../projects_data/190d5889-94f3-4fcb-8735-7b16cd9e7a9b/meshe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
